Commit message: WIP

File: mini_pupper_ws/src/mini_pupper_description/xacro/accessories.xacro (robot description, xacro)
@@ -1,3 +1,27 @@
 <?xml version="1.0"?>
 <robot xmlns:xacro="http://ros.org/wiki/xacro">
+    <xacro:include filename="$(find mini_pupper_description)/xacro/const.xacro" />
+    <xacro:if value="${has_lidar == True}">
+  <link name="lidar">
+    <visual>
+      <origin rpy="0.0 0.0 0.0" xyz="0.0 0.0 0.0"/>
+      <geometry>
+        <mesh filename="package://mini_pupper_description/meshes/lidar.stl"/>
+      </geometry>
+      <material name="black"/>
+    </visual>
+    <collision>
+      <origin rpy="0.0 0.0 0.0" xyz="0.0 0.0 0.0"/>
+      <geometry>
+        <mesh filename="package://mini_pupper_description/meshes/lidar.stl"/>
+      </geometry>
+    </collision>
+  </link>
+  <joint name="base_lidar" type="fixed">
+    <origin rpy="0 0 ${angle_180}" xyz="${lidar_offset_x} 0.0 ${lidar_offset_z}"/>
+    <parent link="base_link"/>
+    <child link="lidar"/>
+    <axis xyz="0 0 0"/>
+  </joint>
+    </xacro:if>
 </robot>

File: mini_pupper_ws/src/mini_pupper_description/xacro/const.xacro (robot description, xacro)
@@ -6,5 +6,11 @@
 -->
 <robot xmlns:xacro="http://www.ros.org/wiki/xacro">
+    <xacro:property name="has_lidar" value="True"/>
+    <xacro:property name="lidar_offset_x" value="-0.01"/>
+    <xacro:property name="lidar_offset_z" value="0.06"/>
+    <xacro:property name="has_oakd" value="False"/>
     <xacro:property name="right_angle" value="1.57079"/>
+    <xacro:property name="angle_135" value="2.35619"/>
+    <xacro:property name="angle_180" value="3.14159"/>
     <xacro:property name="abd_offset_x" value="0.059"/>
     <xacro:property name="abd_offset_y" value="0.0235"/>

File: mini_pupper_ws/src/mini_pupper_description/xacro/leg.xacro (robot description, xacro)
@@ -83,5 +83,5 @@
             <parent link="${name}-pod"/>
             <child link="${name}-femur"/>
-	    <origin rpy="-${right_angle} ${right_angle} 0" xyz="0.0 ${side_sign}${hip_offset_y} 0.0"/>
+	    <origin rpy="-${right_angle} -${angle_135} 0.0" xyz="0.0 ${side_sign}${hip_offset_y} 0.0"/>
             <axis xyz="0 0 1"/>
             <limit lower="0.0" upper="3.4" effort="100" velocity="1000"/>
@@ -90,5 +90,5 @@
             <parent link="${name}-femur"/>
             <child link="${name}-tibia"/>
-	    <origin rpy="0.0 0.0 0.0" xyz="${knee_offset_x} 0.0 ${side_sign}${knee_offset_z}"/>
+	    <origin rpy="0.0 0.0 -${right_angle}" xyz="${knee_offset_x} 0.0 ${side_sign}${knee_offset_z}"/>
             <axis xyz="0 0 1"/>
             <limit lower="-2.8" upper="0.0" effort="100" velocity="1000"/>
