Commit message: WIP

File: mini_pupper_ws/src/mini_pupper_description/xacro/const.xacro (robot description, xacro)
@@ -7,4 +7,5 @@
 <robot xmlns:xacro="http://www.ros.org/wiki/xacro">
     <xacro:property name="has_lidar" value="True"/>
+    <xacro:property name="has_imu" value="True"/>
     <xacro:property name="lidar_offset_x" value="-0.01"/>
     <xacro:property name="lidar_offset_z" value="0.06"/>

File: mini_pupper_ws/src/mini_pupper_description/xacro/imu.xacro (robot description, xacro)
@@ -2,11 +2,11 @@
 <robot xmlns:xacro="http://ros.org/wiki/xacro">
     <xacro:include filename="$(find mini_pupper_description)/xacro/const.xacro" />
-    <xacro:macro name="accessories">
-    <xacro:if value="${has_lidar == True}">
-  <link name="lidar">
+    <xacro:macro name="imu">
+    <xacro:if value="${has_imu == True}">
+  <link name="imu">
     <visual>
       <origin rpy="0.0 0.0 0.0" xyz="0.0 0.0 0.0"/>
       <geometry>
-        <mesh filename="package://mini_pupper_description/meshes/lidar.stl"/>
+        <box size="0.0 0.0 0.0" />
       </geometry>
       <material name="black"/>
@@ -15,13 +15,13 @@
       <origin rpy="0.0 0.0 0.0" xyz="0.0 0.0 0.0"/>
       <geometry>
-        <mesh filename="package://mini_pupper_description/meshes/lidar.stl"/>
+        <box size="0.0 0.0 0.0" />
       </geometry>
     </collision>
   </link>
-  <joint name="base_lidar" type="fixed">
-    <origin rpy="0 0 ${angle_180}" xyz="${lidar_offset_x} 0.0 ${lidar_offset_z}"/>
+  <joint name="base_imu" type="fixed">
+   <origin rpy="0.0 0.0 0.0" xyz="0.0 0.0 0.0"/>
     <parent link="base_link"/>
-    <child link="lidar"/>
-    <axis xyz="0 0 0"/>
+    <child link="imu"/>
+    <axis xyz="0.0 0.0 0.0"/>
   </joint>
     </xacro:if>

File: mini_pupper_ws/src/mini_pupper_description/xacro/mini_pupper_description.xacro (robot description, xacro)
@@ -12,5 +12,8 @@
 <robot name="mini_pupper" xmlns:xacro="http://ros.org/wiki/xacro">
   <xacro:include filename="$(find mini_pupper_description)/xacro/materials.xacro" />
+  <xacro:include filename="$(find mini_pupper_description)/xacro/body.xacro" />
   <xacro:include filename="$(find mini_pupper_description)/xacro/leg.xacro" />
+  <xacro:include filename="$(find mini_pupper_description)/xacro/accessories.xacro" />
+  <xacro:include filename="$(find mini_pupper_description)/xacro/imu.xacro" />
     <!--
     ############################################
@@ -18,39 +21,5 @@
     ############################################
     -->
-    <!--
-    ********************************************
-    ******              PARTS             ******
-    ********************************************
-    -->
-    <link name="base_link">
-        <!--body-->
-        <visual>
-            <geometry>
-                <mesh filename="package://mini_pupper_description/meshes/base_link.stl" scale="1.0 1.0 1.0"/>
-            </geometry>
-            <origin rpy="0 0 0" xyz="0 0 -0.017"/>
-            <material name="white"/>
-        </visual>
-        <collision>
-            <geometry>
-                <box size="0.180 0.060 0.045"/>
-            </geometry>
-            <origin rpy="0 0 0" xyz="0.008 0 0.005"/>
-        </collision>
-        <!--body-battery-holder-->
-        <visual>
-            <geometry>
-                <box size="0.150 0.036 0.008"/>
-            </geometry>
-            <origin rpy="0 0 0" xyz="0.0 0.0 -0.020"/>
-            <material name="black"/>
-        </visual>
-        <collision>
-            <geometry>
-                <box size="0.150 0.036 0.008"/>
-            </geometry>
-            <origin rpy="0 0 0" xyz="0.0 0.0 -0.020"/>
-        </collision>
-    </link>
+    <xacro:body />
     <!--
     ############################################
@@ -61,5 +30,5 @@
     <!--
     ############################################
-    ######              LEG Front Left   ######
+    ######              LEG Front Left    ######
     ############################################
     -->
@@ -67,5 +36,5 @@
     <!--
     ############################################
-    ######              LEG Rear Right   ######
+    ######              LEG Rear Right    ######
     ############################################
     -->
@@ -73,5 +42,5 @@
     <!--
     ############################################
-    ######              Leg Rear Left    ######
+    ######              LEG Rear Left     ######
     ############################################
     -->
@@ -79,7 +48,13 @@
     <!--
     ############################################
+    ######               IMU              ######
+    ############################################
+    -->
+    <xacro:imu />
+    <!--
+    ############################################
     ######               Accessories      ######
     ############################################
     -->
-    <xacro:include filename="$(find mini_pupper_description)/xacro/accessories.xacro" />
+    <xacro:accessories />
 </robot>

Commit message: WIP

File: mini_pupper_ws/src/mini_pupper_description/xacro/const.xacro (robot description, xacro)
@@ -11,4 +11,5 @@
     <xacro:property name="lidar_offset_z" value="0.06"/>
     <xacro:property name="has_oakd" value="False"/>
+    <xacro:property name="angle_45" value="0.785398"/>
     <xacro:property name="right_angle" value="1.57079"/>
     <xacro:property name="angle_135" value="2.35619"/>

File: mini_pupper_ws/src/mini_pupper_description/xacro/leg.xacro (robot description, xacro)
@@ -85,5 +85,5 @@
 	    <origin rpy="-${right_angle} -${angle_135} 0.0" xyz="0.0 ${side_sign}${hip_offset_y} 0.0"/>
             <axis xyz="0 0 1"/>
-            <limit lower="0.0" upper="3.4" effort="100" velocity="1000"/>
+            <limit lower="-${angle_45}" upper="${angle_45}" effort="100" velocity="1000"/>
         </joint>
         <joint name="${name}-knee" type="revolute">
@@ -92,5 +92,5 @@
 	    <origin rpy="0.0 0.0 -${right_angle}" xyz="${knee_offset_x} 0.0 ${side_sign}${knee_offset_z}"/>
             <axis xyz="0 0 1"/>
-            <limit lower="-2.8" upper="0.0" effort="100" velocity="1000"/>
+            <limit lower="-${angle_45}" upper="${angle_45}" effort="100" velocity="1000"/>
         </joint>
         <joint name="${name}-foot" type="fixed">

Commit message: WIP

File: mini_pupper_ws/src/mini_pupper_description/xacro/const.xacro (robot description, xacro)
@@ -8,4 +8,5 @@
     <xacro:property name="has_lidar" value="True"/>
     <xacro:property name="has_imu" value="True"/>
+    <xacro:property name="has_camera" value="True"/>
     <xacro:property name="lidar_offset_x" value="-0.01"/>
     <xacro:property name="lidar_offset_z" value="0.06"/>

File: mini_pupper_ws/src/mini_pupper_description/xacro/lidar.xacro (robot description, xacro)
@@ -2,5 +2,5 @@
 <robot xmlns:xacro="http://ros.org/wiki/xacro">
     <xacro:include filename="$(find mini_pupper_description)/xacro/const.xacro" />
-    <xacro:macro name="accessories">
+    <xacro:macro name="lidar">
     <xacro:if value="${has_lidar == True}">
   <link name="lidar">

File: mini_pupper_ws/src/mini_pupper_description/xacro/mini_pupper_description.xacro (robot description, xacro)
@@ -14,6 +14,7 @@
   <xacro:include filename="$(find mini_pupper_description)/xacro/body.xacro" />
   <xacro:include filename="$(find mini_pupper_description)/xacro/leg.xacro" />
-  <xacro:include filename="$(find mini_pupper_description)/xacro/accessories.xacro" />
+  <xacro:include filename="$(find mini_pupper_description)/xacro/lidar.xacro" />
   <xacro:include filename="$(find mini_pupper_description)/xacro/imu.xacro" />
+  <xacro:include filename="$(find mini_pupper_description)/xacro/camera.xacro" />
     <!--
     ############################################
@@ -54,7 +55,13 @@
     <!--
     ############################################
-    ######               Accessories      ######
+    ######               Lidar LD06       ######
     ############################################
     -->
-    <xacro:accessories />
+    <xacro:lidar />
+    <!--
+    ############################################
+    ######               RPi camera       ######
+    ############################################
+    -->
+    <xacro:camera />
 </robot>
